File: SolarZisterne_PCB.kicad_pcb (KiCad board)
At the start: 2 copper layers, 26 parts, among them J1 Erzeugung, J2 Verbrauch, J3 Solar, J4 Akku, J5 Ultraschall Sensor, J6 Externer Temperatur Sensor, J7 Interner Temperatur Sensor, J8 Erweiterung, U1 MCP1700T-3302E/MB, U2 MCP73871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

Commit message: weiter gearbeite
Parts:
- U2: footprint Housings_DIP:DIP-18_W7.62mm_LongPads -> Housings_DFN_QFN:QFN-20-1EP_4x4mm_Pitch0.5mm
- U4: footprint Housings_DFN_QFN:QFN-20-1EP_4x4mm_Pitch0.5mm -> Housings_DIP:DIP-18_W7.62mm_LongPads
- moved J4 65.4 mm to (167.6, 44.5), turned to 0 degrees
- moved U2 33.0 mm to (170.2, 61.0), turned to 270 degrees
- moved U4 31.1 mm to (135.9, 63.5)
- moved J7 4.58 mm to (102.9, 83.8)
- moved J8 3.59 mm to (108.0, 41.9)
- moved C2 2.54 mm to (172.7, 102.9), turned to 270 degrees
Connections:
- U3 pad 1: (no net) -> Net-(U3-Pad1)
- U3 pad 12: (no net) -> Net-(U3-Pad12)
- U3 pad 13: (no net) -> Net-(U3-Pad13)
- U3 pad 14: (no net) -> Net-(U3-Pad14)
- U3 pad 15: (no net) -> Net-(U3-Pad15)
- U3 pad 7: (no net) -> Net-(U3-Pad7)
- U3 pad 8: (no net) -> Net-(U3-Pad8)
- U4 pad 8: (no net) -> Net-(U4-Pad8)
Routing:
- net GND: track 57.9 -> 152.8 mm
- net +3V3: track 19.4 -> 50.9 mm
- net Net-(C1-Pad1): track 41.0 -> 56.1 mm
- net VCC: track 14.8 -> 0.00 mm
- net (no net): track 0.00 -> 14.8 mm
- net /SDA: track 77.0 -> 81.5 mm
- net /SCL: track 86.9 -> 90.0 mm
