File: KiCAD PCB/SolarZisterne_PCB.sch (KiCad schematic (older format))
At the start: 26 parts, among them J1 Erzeugung, J2 Verbrauch, J3 Solar, J4 Akku, J5 Ultraschall Sensor, J6 Externer Temperatur Sensor, J7 Interner Temperatur Sensor, J8 Erweiterung, U1 MCP1700T-3302E/MB, U2 MCP73871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

Commit message: Sicherung bevor die Messung mit den DHT22 Sensoren entfernt wird
Parts:
- J3, J4: footprint Connectors_Terminal_Blocks:TerminalBlock_Pheonix_MKDS1.5-2pol -> Connectors_Terminal_Blocks:TerminalBlock_Pheonix_PT-3.5mm_2pol
- J5: footprint Connectors_Terminal_Blocks:TerminalBlock_Pheonix_MKDS1.5-4pol -> Connectors_Terminal_Blocks:TerminalBlock_Pheonix_PT-3.5mm_4pol
Other:
- note added: "Graund mit Jumper für GPIO"
Changed lines of the file:
@@
 F 0 "J3" H 850 1700 50  0000 C TNN
 F 1 "Solar" V 700 1450 50  0000 C TNN
-F 2 "Connectors_Terminal_Blocks:TerminalBlock_Pheonix_MKDS1.5-2pol" H 850 1225 50  0001 C CNN
+F 2 "Connectors_Terminal_Blocks:TerminalBlock_Pheonix_PT-3.5mm_2pol" H 850 1225 50  0001 C CNN
 F 3 "" H 825 1450 50  0001 C CNN
 	1    850  1450
@@
 F 0 "J4" H 7000 2150 50  0000 C TNN
 F 1 "Akku" V 6850 1900 50  0000 C TNN
-F 2 "Connectors_Terminal_Blocks:TerminalBlock_Pheonix_MKDS1.5-2pol" H 7000 1675 50  0001 C CNN
+F 2 "Connectors_Terminal_Blocks:TerminalBlock_Pheonix_PT-3.5mm_2pol" H 7000 1675 50  0001 C CNN
 F 3 "" H 6975 1900 50  0001 C CNN
 	1    7000 1900
@@
 F 0 "J5" H 7350 4750 50  0000 C TNN
 F 1 "Ultraschall Sensor" V 7200 4300 50  0000 C TNN
-F 2 "Connectors_Terminal_Blocks:TerminalBlock_Pheonix_MKDS1.5-4pol" H 7350 3875 50  0001 C CNN
+F 2 "Connectors_Terminal_Blocks:TerminalBlock_Pheonix_PT-3.5mm_4pol" H 7350 3875 50  0001 C CNN
 F 3 "" H 7325 4500 50  0001 C CNN
 	1    7350 4300
@@
 Wire Wire Line
 	10750 900  10750 800
+Text Notes 9700 5250 0    60   ~ 0
+Graund mit Jumper für GPIO
 $EndSCHEMATC

Commit message: Before Änderung Ultraschall
Other:
- note added: "gegen 6pol austauschen"
- note added: "gegen 6pol austauschen\nplus VCC"
Changed lines of the file:
@@
 Text Notes 9700 5250 0    60   ~ 0
 Graund mit Jumper für GPIO
+Text Notes 7750 4950 0    60   ~ 0
+gegen 6pol austauschen
+Text Notes 9050 5050 0    60   ~ 0
+gegen 6pol austauschen\nplus VCC
 $EndSCHEMATC

Commit message: PCB Update
Parts:
- removed J7: Interner Temperatur Sensor, Pin_Headers:Pin_Header_Straight_1x04_Pitch2.54mm, symbol CONN_01X04
- added J10, J11, J12, J13, J9: GS2, Connectors:GS2, symbol GS2
- added J7: Interner Temperatur Sensor, Pin_Headers:Pin_Header_Straight_1x06_Pitch2.54mm, symbol CONN_01X06
- J6: footprint Connectors_Terminal_Blocks:TerminalBlock_Pheonix_MKDS1.5-4pol -> Connectors_Terminal_Blocks:TerminalBlock_Pheonix_PT-3.5mm_4pol
Connections:
- net +3V3: now also J7.1 (P1), J7.6 (P6)
- net Echo: now also U3.6 (D1); no longer U3.3 (D4)
- net GND: now also J10.2 (G2), J11.2 (G2), J12.2 (G2), J13.2 (G2), J7.2 (P2), J9.2 (G2)
- net GPB3: now also J9.1 (G1)
- net GPB4: now also J10.1 (G1)
- net GPB5: now also J11.1 (G1)
- net GPB6: now also J12.1 (G1)
- net GPB7: now also J13.1 (G1)
- net SCL: now also U3.3 (D4), J7.3 (P3); no longer U3.6 (D1)
- net SDA: now also U3.4 (D3), J7.4 (P4); no longer U3.5 (D2)
- net Trig: now also U3.5 (D2); no longer U3.4 (D3)
- no-connect marks 8 -> 9
Other:
- note added: "Pins D5, D6, D7, D8 werden durch SD Karte benutzt\nPins D1, D2 für Ultraschallsensor\nPins D3, D4 werden für I2C Sensoren benutzt\nI2C brauch keine Pull-Up Wiederstand die sind\nschon bei den Temp. Sensoren drin.\n"
- note removed: "Graund mit Jumper für GPIO"
- note removed: "Pins D5, D6, D7, D8 werden durch SD Karte beansprucht\nPins D2, D1 werden für I2C Sensoren benutzt\nPins D3, D4 für Ultraschallsensor"
- note removed: "SDA\nSCL"
- note removed: "bracuh wahrscheinlich\nnoch Pull-Up"
- note removed: "gegen 6pol austauschen"
- note removed: "gegen 6pol austauschen\nplus VCC"
- moved on the sheet: J5, J6, J8

Commit message: PCB update
Parts:
- removed C3: 4.7uF, Capacitors_THT:C_Disc_D5.0mm_W2.5mm_P2.50mm, symbol C
- removed C4: 1uF, Capacitors_THT:C_Disc_D5.0mm_W2.5mm_P2.50mm, symbol C
- removed U1: MCP1700T-3302E/MB, TO_SOT_Packages_THT:TO-92_Inline_Narrow_Oval, symbol MCP1700T-3002E/TT
- added J14: Buck-Conv D24V5F3, Pin_Headers:Pin_Header_Straight_1x04_Pitch2.54mm, symbol CONN_01X04
Connections:
- net +3V3: now also J14.1 (P1)
- net GND: now also J4.2, J14.2 (P2), J14.4 (P4); no longer J4.1
- net at C5.1, U2.14 (VBAT), U2.15 (VBAT)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: now also J4.1; no longer J4.2
- net at J2.5 (P5): now also J14.3 (P3)
Other:
- moved on the sheet: J4

Commit message: fast aller Leiterbahnen
Parts:
- U3: value WeMos_mini -> WeMos_Mini
Changed lines of the file:
@@
 P 2300 4350
 F 0 "U3" H 2300 4850 60  0000 C CNN
-F 1 "WeMos_mini" H 2300 3850 60  0000 C CNN
+F 1 "WeMos_Mini" H 2300 3850 60  0000 C CNN
 F 2 "wemos_d1_mini:D1_mini_board" H 2850 3650 60  0001 C CNN
 F 3 "" H 2850 3650 60  0000 C CNN
@@
 $EndComp
 $Comp
-L GND #PWR015
+L GND #PWR014
 U 1 1 595425EA
 P 6550 2250
-F 0 "#PWR015" H 6550 2000 50  0001 C CNN
+F 0 "#PWR014" H 6550 2000 50  0001 C CNN
 F 1 "GND" H 6550 2100 50  0000 C CNN
 F 2 "" H 6550 2250 50  0001 C CNN
@@
 $EndComp
 $Comp
-L +3.3V #PWR016
+L +3.3V #PWR015
 U 1 1 59544F20
 P 2950 3900
-F 0 "#PWR016" H 2950 3750 50  0001 C CNN
+F 0 "#PWR015" H 2950 3750 50  0001 C CNN
 F 1 "+3.3V" H 2950 4040 50  0000 C CNN
 F 2 "" H 2950 3900 50  0001 C CNN
@@
 $EndComp
 $Comp
-L GND #PWR017
+L GND #PWR016
 U 1 1 595451B9
 P 1300 4150
-F 0 "#PWR017" H 1300 3900 50  0001 C CNN
+F 0 "#PWR016" H 1300 3900 50  0001 C CNN
 F 1 "GND" H 1300 4000 50  0000 C CNN
 F 2 "" H 1300 4150 50  0001 C CNN
@@
 $EndComp
 $Comp
-L GND #PWR018
+L GND #PWR017
 U 1 1 5954691E
 P 1850 900
-F 0 "#PWR018" H 1850 650 50  0001 C CNN
+F 0 "#PWR017" H 1850 650 50  0001 C CNN
 F 1 "GND" H 1850 750 50  0000 C CNN
 F 2 "" H 1850 900 50  0001 C CNN
@@
 $EndComp
 $Comp
-L +3.3V #PWR019
+L +3.3V #PWR018
 U 1 1 59547AC5
 P 2150 700
-F 0 "#PWR019" H 2150 550 50  0001 C CNN
+F 0 "#PWR018" H 2150 550 50  0001 C CNN
 F 1 "+3.3V" H 2150 840 50  0000 C CNN
 F 2 "" H 2150 700 50  0001 C CNN
@@
 $EndComp
 $Comp
-L +3.3V #PWR020
+L +3.3V #PWR019
 U 1 1 595489A4
 P 6450 950
-F 0 "#PWR020" H 6450 800 50  0001 C CNN
+F 0 "#PWR019" H 6450 800 50  0001 C CNN
 F 1 "+3.3V" H 6450 1090 50  0000 C CNN
 F 2 "" H 6450 950 50  0001 C CNN
@@
 $EndComp
 $Comp
-L GND #PWR021
+L GND #PWR020
 U 1 1 59548AB7
 P 5850 1150
-F 0 "#PWR021" H 5850 900 50  0001 C CNN
+F 0 "#PWR020" H 5850 900 50  0001 C CNN
 F 1 "GND" H 5850 1000 50  0000 C CNN
 F 2 "" H 5850 1150 50  0001 C CNN
@@
 SDA
 $Comp
-L +3.3V #PWR022
+L +3.3V #PWR021
 U 1 1 5954B7EF
 P 4850 3650
-F 0 "#PWR022" H 4850 3500 50  0001 C CNN
+F 0 "#PWR021" H 4850 3500 50  0001 C CNN
 F 1 "+3.3V" H 4850 3790 50  0000 C CNN
 F 2 "" H 4850 3650 50  0001 C CNN
@@
 $EndComp
 $Comp
-L GND #PWR023
+L GND #PWR022
 U 1 1 5954B8BD
 P 4850 5150
-F 0 "#PWR023" H 4850 4900 50  0001 C CNN
+F 0 "#PWR022" H 4850 4900 50  0001 C CNN
 F 1 "GND" H 4850 5000 50  0000 C CNN
 F 2 "" H 4850 5150 50  0001 C CNN
@@
 $EndComp
 $Comp
-L +3.3V #PWR024
+L +3.3V #PWR023
 U 1 1 5954DD9B
 P 6300 3950
-F 0 "#PWR024" H 6300 3800 50  0001 C CNN
+F 0 "#PWR023" H 6300 3800 50  0001 C CNN
 F 1 "+3.3V" H 6300 4090 50  0000 C CNN
 F 2 "" H 6300 3950 50  0001 C CNN
@@
 $EndComp
 $Comp
-L GND #PWR025
+L GND #PWR024
 U 1 1 5954DDEB
 P 6300 4750
-F 0 "#PWR025" H 6300 4500 50  0001 C CNN
+F 0 "#PWR024" H 6300 4500 50  0001 C CNN
 F 1 "GND" H 6300 4600 50  0000 C CNN
 F 2 "" H 6300 4750 50  0001 C CNN
@@
 $EndComp
 $Comp
-L +3.3V #PWR026
+L +3.3V #PWR025
 U 1 1 5955031D
 P 10600 3900
-F 0 "#PWR026" H 10600 3750 50  0001 C CNN
+F 0 "#PWR025" H 10600 3750 50  0001 C CNN
 F 1 "+3.3V" H 10600 4040 50  0000 C CNN
 F 2 "" H 10600 3900 50  0001 C CNN
@@
 $EndComp
 $Comp
-L GND #PWR027
+L GND #PWR026
 U 1 1 59550430
 P 10600 4900
-F 0 "#PWR027" H 10600 4650 50  0001 C CNN
+F 0 "#PWR026" H 10600 4650 50  0001 C CNN
 F 1 "GND" H 10600 4750 50  0000 C CNN
 F 2 "" H 10600 4900 50  0001 C CNN
@@
 $EndComp
 $Comp
-L +3.3V #PWR028
+L +3.3V #PWR027
 U 1 1 5956BC5D
 P 7200 3950
-F 0 "#PWR028" H 7200 3800 50  0001 C CNN
+F 0 "#PWR027" H 7200 3800 50  0001 C CNN
 F 1 "+3.3V" H 7200 4090 50  0000 C CNN
 F 2 "" H 7200 3950 50  0001 C CNN
@@
 $EndComp
 $Comp
-L GND #PWR029
+L GND #PWR028
 U 1 1 5956BCB3
 P 6900 4300
-F 0 "#PWR029" H 6900 4050 50  0001 C CNN
+F 0 "#PWR028" H 6900 4050 50  0001 C CNN
 F 1 "GND" H 6900 4150 50  0000 C CNN
 F 2 "" H 6900 4300 50  0001 C CNN
@@
 SDA
 $Comp
-L +3.3V #PWR030
+L +3.3V #PWR029
 U 1 1 5956C1F1
 P 7850 4050
-F 0 "#PWR030" H 7850 3900 50  0001 C CNN
+F 0 "#PWR029" H 7850 3900 50  0001 C CNN
 F 1 "+3.3V" H 7850 4190 50  0000 C CNN
 F 2 "" H 7850 4050 50  0001 C CNN
@@
 $EndComp
 $Comp
-L GND #PWR031
+L GND #PWR030
 U 1 1 5956C24A
 P 7950 4300
-F 0 "#PWR031" H 7950 4050 50  0001 C CNN
+F 0 "#PWR030" H 7950 4050 50  0001 C CNN
 F 1 "GND" H 7950 4150 50  0000 C CNN
 F 2 "" H 7950 4300 50  0001 C CNN
@@
 SDA
 $Comp
-L PWR_FLAG #FLG032
+L PWR_FLAG #FLG031
 U 1 1 59581FAF
 P 10750 800
-F 0 "#FLG032" H 10750 875 50  0001 C CNN
+F 0 "#FLG031" H 10750 875 50  0001 C CNN
 F 1 "PWR_FLAG" H 10750 950 50  0000 C CNN
 F 2 "" H 10750 800 50  0001 C CNN
@@
 $EndComp
 $Comp
-L GND #PWR033
+L GND #PWR032
 U 1 1 59582029
 P 10750 900
-F 0 "#PWR033" H 10750 650 50  0001 C CNN
+F 0 "#PWR032" H 10750 650 50  0001 C CNN
 F 1 "GND" H 10750 750 50  0000 C CNN
 F 2 "" H 10750 900 50  0001 C CNN
@@
 $EndComp
 $Comp
-L GND #PWR034
+L GND #PWR033
 U 1 1 5973F0E8
 P 10250 5150
-F 0 "#PWR034" H 10250 4900 50  0001 C CNN
+F 0 "#PWR033" H 10250 4900 50  0001 C CNN
 F 1 "GND" H 10250 5000 50  0000 C CNN
 F 2 "" H 10250 5150 50  0001 C CNN
@@
 $EndComp
 $Comp
-L GND #PWR035
+L GND #PWR034
 U 1 1 5973F14D
 P 9950 5150
-F 0 "#PWR035" H 9950 4900 50  0001 C CNN
+F 0 "#PWR034" H 9950 4900 50  0001 C CNN
 F 1 "GND" H 9950 5000 50  0000 C CNN
 F 2 "" H 9950 5150 50  0001 C CNN
@@
 $EndComp
 $Comp
-L GND #PWR036
+L GND #PWR035
 U 1 1 5973F1B2
 P 9650 5150
-F 0 "#PWR036" H 9650 4900 50  0001 C CNN
+F 0 "#PWR035" H 9650 4900 50  0001 C CNN
 F 1 "GND" H 9650 5000 50  0000 C CNN
 F 2 "" H 9650 5150 50  0001 C CNN
@@
 $EndComp
 $Comp
-L GND #PWR037
+L GND #PWR036
 U 1 1 5973F217
 P 9300 5150
-F 0 "#PWR037" H 9300 4900 50  0001 C CNN
+F 0 "#PWR036" H 9300 4900 50  0001 C CNN
 F 1 "GND" H 9300 5000 50  0000 C CNN
 F 2 "" H 9300 5150 50  0001 C CNN
@@
 $EndComp
 $Comp
-L GND #PWR038
+L GND #PWR037
 U 1 1 5973F59A
 P 8950 5150
-F 0 "#PWR038" H 8950 4900 50  0001 C CNN
+F 0 "#PWR037" H 8950 4900 50  0001 C CNN
 F 1 "GND" H 8950 5000 50  0000 C CNN
 F 2 "" H 8950 5150 50  0001 C CNN
@@
 $EndComp
 $Comp
-L GND #PWR039
+L GND #PWR038
 U 1 1 5974ECAC
 P 7500 1800
-F 0 "#PWR039" H 7500 1550 50  0001 C CNN
+F 0 "#PWR038" H 7500 1550 50  0001 C CNN
 F 1 "GND" H 7500 1650 50  0000 C CNN
 F 2 "" H 7500 1800 50  0001 C CNN
@@
 Connection ~ 7500 1700
 $Comp
-L +3.3V #PWR040
+L +3.3V #PWR039
 U 1 1 5974EF13
 P 7500 1300
-F 0 "#PWR040" H 7500 1150 50  0001 C CNN
+F 0 "#PWR039" H 7500 1150 50  0001 C CNN
 F 1 "+3.3V" H 7500 1440 50  0000 C CNN
 F 2 "" H 7500 1300 50  0001 C CNN
